Commit message: fix urdf

File: pkg_techfest_imc/urdf/micromouse_robot1.urdf (robot description, URDF)
Before this commit: robot my_mm_robot, 4 links, 3 joints
Links:
- link link_chassis: geometry collision box size=0.07 0.07 0.02; collision sphere radius=0.003
- link link_left_wheel: geometry collision cylinder length=0.007 radius=0.0175; visual cylinder length=0.007 radius=0.0175
- link link_right_wheel: geometry collision cylinder length=0.007 radius=0.0175; visual cylinder length=0.007 radius=0.0175
- link sensor_laser: mass 0 -> 0.4; geometry collision cylinder length=0.022 radius=0.005; visual cylinder length=0.022 radius=0.005
Joints:
- joint joint_left_wheel: origin xyz=${Factor*0.028} ${Factor*0.02} 0 rpy=0 0 0 -> xyz=0.028 0.02 0 rpy=0 0 0
- joint joint_right_wheel: axis ${Factor*1} 0 0 -> 1 0 0; origin xyz=${Factor*(-0.03)}  ${Factor*0.02}    0 rpy=0 0 0 -> xyz=-0.03  0.02    0 rpy=0 0 0
- joint joint_sensor_laser: origin xyz=0    0    ${Factor*0.018} rpy=0  0  -1.57 -> xyz=0    0    0.018 rpy=0  0  -1.57
